Commit message: Fun fact: making a chess bot with 4 dof arm is a pain in the arse.

File: chessaton_description/urdf/chessaton.urdf (robot description, URDF)
Before this commit: robot chessaton, 9 links, 8 joints
Links:
- added link virtual_roll_link, mass 1.0e-03; visual box size=0.01 0.01 0.01
- added link virtual_yaw_link, mass 1.0e-03; visual box size=0.01 0.01 0.01
Joints:
- added joint virtual_roll_joint: type revolute, parent chessaton_link4, child virtual_roll_link, origin xyz=0.072842 -0.034194 -0.0048547 rpy=0 0 0, axis 1 0 0, limit lower=-3.1415 upper=3.1415 effort=54.0 velocity=3.14
- added joint virtual_yaw_joint: type revolute, parent virtual_roll_link, child virtual_yaw_link, origin xyz=0.0 0.0 0.0 rpy=0 0 0, axis 0 0 1, limit lower=-3.1415 upper=3.1415 effort=54.0 velocity=3.14
- joint gripper_joint: origin xyz=0.072842 -0.034194 -0.0048547 rpy=0 0 0 -> xyz=0.0 0.0 0.0 rpy=0 0 0; parent chessaton_link4 -> virtual_yaw_link

File: chessaton_description/urdf/chessaton.urdf.xacro (robot description, xacro)
@@ -196,9 +196,65 @@
         </inertial>
 	</link>
-	<joint name="gripper_joint" type="fixed">
-	  <origin xyz="0.072842 -0.034194 -0.0048547" rpy="0 0 0" />
-	  <parent link="chessaton_link4" />
-	  <child link="chessaton_gripper" />
-	  <axis xyz="0 0 0" />
+    <!-- Virtual roll joint -->
+    <joint name="virtual_roll_joint" type="revolute">
+      <limit lower="-3.1415" upper="3.1415" effort="54.0" velocity="3.14"/>
+      <parent link="chessaton_link4"/>
+      <child link="virtual_roll_link"/>
+      <axis xyz="1 0 0"/>
+      <origin xyz="0.072842 -0.034194 -0.0048547" rpy="0 0 0"/>
+      <dynamics damping="0.0" friction="0.0"/>
+    </joint>
+    <!-- Virtual roll link -->
+    <link name="virtual_roll_link">
+      <visual>
+        <origin xyz="0 0 0" rpy="0 0 0"/>
+        <geometry>
+          <box size="0.01 0.01 0.01" />
+        </geometry>
+       </visual>
+      <inertial>
+        <origin xyz="0 0 0" />
+        <mass value="1.0e-03" />
+        <inertia ixx="1.0e-03" ixy="0.0" ixz="0.0"
+                 iyy="1.0e-03" iyz="0.0"
+                 izz="1.0e-03" />
+      </inertial>
+    </link>
+    <!-- Virtual yaw joint -->
+    <joint name="virtual_yaw_joint" type="revolute">
+      <limit lower="-3.1415" upper="3.1415" effort="54.0" velocity="3.14"/>
+      <parent link="virtual_roll_link"/>
+      <child link="virtual_yaw_link"/>
+      <axis xyz="0 0 1"/>
+      <origin xyz="0.0 0.0 0.0" rpy="0 0 0"/>
+      <dynamics damping="0.0" friction="0.0"/>
+    </joint>
+    <!-- Virtual yaw link -->
+    <link name="virtual_yaw_link">
+      <visual>
+        <origin xyz="0 0 0" rpy="0 0 0"/>
+        <geometry>
+          <box size="0.01 0.01 0.01" />
+        </geometry>
+       </visual>
+      <inertial>
+        <origin xyz="0 0 0" />
+        <mass value="1.0e-03" />
+        <inertia ixx="1.0e-03" ixy="0.0" ixz="0.0"
+                 iyy="1.0e-03" iyz="0.0"
+                 izz="1.0e-03" />
+      </inertial>
+    </link>
+	<!-- <joint name="gripper_joint" type="fixed"> -->
+	  <!-- <origin xyz="0.072842 -0.034194 -0.0048547" rpy="0 0 0" /> -->
+	  <!-- <parent link="virtual_yaw_link" /> -->
+	  <!-- <child link="chessaton_gripper" /> -->
+	  <!-- <axis xyz="0 0 0" /> -->
+	<!-- </joint> -->
+    <joint name="gripper_joint" type="fixed">
+        <origin xyz="0.0 0.0 0.0" rpy="0 0 0"/>
+	    <parent link="virtual_yaw_link" />
+	    <child link="chessaton_gripper" />
+	    <axis xyz="0 0 0" />
 	</joint>
 	<link name="chessaton_gripper">

File: chessaton_description/urdf/chessaton_gazebo.xacro (robot description, xacro)
@@ -27,4 +27,10 @@
         <material>Gazebo/White</material>
     </gazebo>
+    <gazebo reference="virtual_roll_link">
+        <material>Gazebo/White</material>
+    </gazebo>
+    <gazebo reference="virtual_yaw_link">
+        <material>Gazebo/White</material>
+    </gazebo>
     <!--       -->
     <!-- Macro -->

File: chessaton_moveit_config/srdf/chessaton_macro.srdf.xacro (robot description, xacro)
@@ -17,4 +17,6 @@
             <joint name="chessaton_joint3"/>
             <joint name="chessaton_joint4"/>
+            <joint name="virtual_roll_joint"/>
+            <joint name="virtual_yaw_joint"/>
         </group>
         <group name="chessaton_hand">
@@ -29,4 +31,6 @@
             <joint name="chessaton_joint3" value="0"/>
             <joint name="chessaton_joint4" value="0"/>
+            <joint name="virtual_roll_joint" value="0"/>
+            <joint name="virtual_yaw_joint" value="0"/>
         </group_state>
         <group_state name="hand_close" group="chessaton_hand">
@@ -42,18 +46,33 @@
         <!--DISABLE COLLISIONS- By default it is assumed that any link of the robot could potentially come into collision with any other link in the robot. This tag disables collision checking between a specified pair of links. -->
         <disable_collisions link1="chessaton_gripper" link2="chessaton_link3" reason="Never"/>
-        <disable_collisions link1="chessaton_gripper" link2="chessaton_link4" reason="Adjacent"/>
-        <disable_collisions link1="chessaton_gripper" link2="left_finger" reason="Adjacent"/>
-        <disable_collisions link1="chessaton_gripper" link2="right_finger" reason="Adjacent"/>
-        <disable_collisions link1="chessaton_link0" link2="chessaton_link1" reason="Adjacent"/>
-        <disable_collisions link1="chessaton_link0" link2="chessaton_link2" reason="Never"/>
-        <disable_collisions link1="chessaton_link1" link2="chessaton_link2" reason="Adjacent"/>
-        <disable_collisions link1="chessaton_link1" link2="chessaton_link3" reason="Never"/>
-        <disable_collisions link1="chessaton_link2" link2="chessaton_link3" reason="Adjacent"/>
-        <disable_collisions link1="chessaton_link3" link2="chessaton_link4" reason="Adjacent"/>
-        <disable_collisions link1="chessaton_link3" link2="left_finger" reason="Never"/>
-        <disable_collisions link1="chessaton_link3" link2="right_finger" reason="Never"/>
-        <disable_collisions link1="chessaton_link4" link2="left_finger" reason="Never"/>
-        <disable_collisions link1="chessaton_link4" link2="right_finger" reason="Never"/>
-        <disable_collisions link1="left_finger" link2="right_finger" reason="Never"/>
+  <disable_collisions link1="chessaton_gripper" link2="chessaton_link4" reason="Adjacent"/>
+  <disable_collisions link1="chessaton_gripper" link2="left_finger" reason="Adjacent"/>
+  <disable_collisions link1="chessaton_gripper" link2="right_finger" reason="Adjacent"/>
+  <disable_collisions link1="chessaton_link0" link2="chessaton_link1" reason="Adjacent"/>
+  <disable_collisions link1="chessaton_link0" link2="chessaton_link2" reason="Never"/>
+  <disable_collisions link1="chessaton_link1" link2="chessaton_link2" reason="Adjacent"/>
+  <disable_collisions link1="chessaton_link1" link2="chessaton_link3" reason="Never"/>
+  <disable_collisions link1="chessaton_link2" link2="chessaton_link3" reason="Adjacent"/>
+    <disable_collisions link1="chessaton_link2" link2="virtual_roll_link" reason="Never"/>
+    <disable_collisions link1="chessaton_link2" link2="virtual_yaw_link" reason="Never"/>
+  <disable_collisions link1="chessaton_link3" link2="chessaton_link4" reason="Adjacent"/>
+  <disable_collisions link1="chessaton_link3" link2="left_finger" reason="Never"/>
+  <disable_collisions link1="chessaton_link3" link2="right_finger" reason="Never"/>
+  <disable_collisions link1="chessaton_link4" link2="left_finger" reason="Never"/>
+  <disable_collisions link1="chessaton_link4" link2="right_finger" reason="Never"/>
+  <disable_collisions link1="left_finger" link2="right_finger" reason="Never"/>
+    <disable_collisions link1="chessaton_link3" link2="virtual_roll_link" reason="Never"/>
+    <disable_collisions link1="chessaton_link3" link2="virtual_yaw_link" reason="Never"/>
+    <disable_collisions link1="chessaton_link4" link2="virtual_roll_link" reason="Adjacent"/>
+    <disable_collisions link1="chessaton_link4" link2="virtual_yaw_link" reason="Never"/>
+    <disable_collisions link1="virtual_roll_link" link2="virtual_yaw_link" reason="Adjacent"/>
+    <disable_collisions link1="chessaton_link1" link2="virtual_roll_link" reason="Never"/>
+    <disable_collisions link1="chessaton_link1" link2="virtual_yaw_link" reason="Never"/>
+    <disable_collisions link1="chessaton_gripper" link2="virtual_roll_link" reason="Default"/>
+    <disable_collisions link1="chessaton_gripper" link2="virtual_yaw_link" reason="Adjacent"/>
+    <disable_collisions link1="right_finger" link2="virtual_roll_link" reason="Never"/>
+    <disable_collisions link1="right_finger" link2="virtual_yaw_link" reason="Never"/>
+    <disable_collisions link1="left_finger" link2="virtual_roll_link" reason="Never"/>
+    <disable_collisions link1="left_finger" link2="virtual_yaw_link" reason="Never"/>
     </xacro:macro>
 </robot>

Commit message: Add: add 2 dummy joints (roll and yaw) for gripper's tcp frame

File: chessaton_description/urdf/chessaton.urdf (robot description, URDF)
Before this commit: robot chessaton, 9 links, 8 joints
Links:
- added link chessaton_hand_tcp
- added link chessaton_hand_tcp_roll, mass 0.0088
- added link chessaton_hand_tcp_yaw, mass 0.0088
Joints:
- added joint chessaton_hand_tcp_roll_virtual_joint: type revolute, parent chessaton_gripper, child chessaton_hand_tcp_roll, origin xyz=0.02 0 -0.005 rpy=0 0 0, axis -1 0 0, limit lower=-1.5707963267948966 upper=1.5707963267948966 effort=0 velocity=6
- added joint chessaton_hand_tcp_virtual_joint: type fixed, parent chessaton_hand_tcp_yaw, child chessaton_hand_tcp, origin xyz=0 0 0 rpy=0 0 0
- added joint chessaton_hand_tcp_yaw_virtual_joint: type revolute, parent chessaton_hand_tcp_roll, child chessaton_hand_tcp_yaw, origin xyz=0 0 0 rpy=0 0 0, axis 0 0 -1, limit lower=-1.5707963267948966 upper=1.5707963267948966 effort=0 velocity=6

File: chessaton_description/urdf/chessaton.urdf.xacro (robot description, xacro)
@@ -8,4 +8,5 @@
     <xacro:include filename="$(find chessaton_description)/urdf/chessaton_gazebo.xacro" />
     <xacro:include filename="$(find chessaton_description)/urdf/chessaton.ros2_control" />
+    <xacro:include filename="$(find chessaton_description)/urdf/chessaton_hand.xacro" />
     <!--            -->
     <!-- Parameters -->
@@ -17,4 +18,5 @@
     <!-- Flag to enable default gripper -->
     <xacro:arg name="gripper" default="true" />
+    <xacro:arg name="virtual_dof" default="true" />
     <!-- ros2_control -->
     <!-- Flag to enable ros2 controllers for manipulator -->
@@ -202,101 +204,37 @@
 	  <axis xyz="0 0 0" />
 	</joint>
-	<link name="chessaton_gripper">
-		<visual>
-			<origin xyz="0 0 0" rpy="0 0 0" />
-			<geometry>
-			  <mesh filename="file://$(find chessaton_description)/meshes/chessaton_gripper.STL" />
-			</geometry>
-			<material name="color_gripper" />
-		</visual>
-		<collision>
-			<origin xyz="0 0 0" rpy="0 0 0" />
-			<geometry>
-				<mesh filename="file://$(find chessaton_description)/meshes/chessaton_gripper.STL" />
-			</geometry>
-		</collision>
-        <inertial>
-            <origin xyz="-0.027242 0.0063062 -0.003963" rpy="0 0 0" />
-            <mass value="0.07416" />
-            <inertia
-              ixx="2.5968E-05"
-              ixy="8.488E-08"
-              ixz="-4.236E-07"
-              iyy="1.3082E-05"
-              iyz="-1.6429E-09"
-              izz="2.6136E-05" />
-        </inertial>
-	</link>
-	<joint name="left_finger_joint" type="prismatic">
-		<origin xyz="0 0 0" rpy="0 0 0" />
-		<parent link="chessaton_gripper" />
-		<child link="left_finger" />
-		<axis xyz="0 1 0" />
-		<dynamics damping="1.0" friction="1.0" />
-		<limit lower="0" upper="0.03" effort="100" velocity="0.2" />
-	</joint>
-	<link name="left_finger">
-    	<visual>
-    	  <origin xyz="0 0 0" rpy="0 0 0" />
-    	  <geometry>
-    	    <mesh filename="file://$(find chessaton_description)/meshes/left_finger.STL" />
-    	  </geometry>
-    	  <material name="color_gripper_lfinger" />
-    	</visual>
-    	<collision>
-    	  <origin xyz="0 0 0" rpy="0 0 0" />
-    	  <geometry>
-    	    <mesh filename="file://$(find chessaton_description)/meshes/left_finger.STL" />
-    	  </geometry>
-    	</collision>
-        <inertial>
-            <origin
-              xyz="0.011394 0.0086324 -0.005"
-              rpy="0 0 0" />
-            <mass
-              value="0.0088" />
-            <inertia
-              ixx="6.0646E-07"
-              ixy="1.4141E-07"
-              ixz="2.4551E-21"
-              iyy="9.0397E-07"
-              iyz="-6.5992E-22"
-              izz="8.4377E-07" />
-        </inertial>
-	</link>
-	<joint name="right_finger_joint" type="prismatic">
-		<origin xyz="0 0 0" rpy="0 0 0" />
-		<parent link="chessaton_gripper" />
-		<child link="right_finger" />
-		<axis xyz="0 1 0" />
-		<dynamics damping="1.0" friction="1.0" />
-		<limit lower="-0.03" upper="0" effort="100" velocity="0.2" />
-	</joint>
-	<link name="right_finger">
-		<visual>
-		  <origin xyz="0 0 0" rpy="0 0 0" />
-		  <geometry>
-		    <mesh filename="file://$(find chessaton_description)/meshes/right_finger.STL" />
-		  </geometry>
-		  <material name="color_gripper_rfinger" />
-		</visual>
-		<collision>
-		  <origin xyz="0 0 0" rpy="0 0 0" />
-		  <geometry>
-		    <mesh filename="file://$(find chessaton_description)/meshes/right_finger.STL" />
-		  </geometry>
-		</collision>
-        <inertial>
-            <origin xyz="0.011394 -0.0086324 -0.005" rpy="0 0 0" />
-            <mass value="0.0088" />
-            <inertia
-              ixx="6.0646E-07"
-              ixy="-1.4141E-07"
-              ixz="1.2142E-21"
-              iyy="9.0397E-07"
-              iyz="7.2151E-22"
-              izz="8.4377E-07" />
-        </inertial>
-	</link>
+    <xacro:chessaton_hand
+        virtual_dof="$(arg virtual_dof)"
+    />
+      <!-- Transmission macro -->
+  <!-- <xacro:macro name="SimpleTransmissionPosition" params="joint n">
+    <transmission name="tran${n}">
+      <type>transmission_interface/SimpleTransmission</type>
+      <joint name="${joint}">
+        <hardwareInterface>hardware_interface/PositionJointInterface</hardwareInterface>
+      </joint>
+      <actuator name="motor${n}">
+        <mechanicalReduction>1</mechanicalReduction>
+      </actuator>
+    </transmission>
+  </xacro:macro> -->
+  <!-- Transmission macro -->
+  <!-- <xacro:macro name="SimpleTransmissionEffort" params="joint n">
+    <transmission name="tran${n}">
+      <type>transmission_interface/SimpleTransmission</type>
+      <joint name="${joint}">
+        <hardwareInterface>hardware_interface/EffortJointInterface</hardwareInterface>
+      </joint>
+      <actuator name="motor${n}">
+        <mechanicalReduction>1</mechanicalReduction>
+      </actuator>
+    </transmission>
+  </xacro:macro> -->
+  <!-- <xacro:SimpleTransmissionEffort n="1" joint="chessaton_joint1" />
+  <xacro:SimpleTransmissionEffort n="2" joint="chessaton_joint2" />
+  <xacro:SimpleTransmissionEffort n="3" joint="chessaton_joint3" />
+  <xacro:SimpleTransmissionEffort n="4" joint="chessaton_joint4" />
+  <xacro:SimpleTransmissionEffort n="5" joint="left_finger_joint" />
+  <xacro:SimpleTransmissionEffort n="6" joint="right_finger_joint" /> -->
     <xacro:gz_ros2_control
         ros2_controller_parameters="$(arg ros2_controller_parameters)"

File: chessaton_description/urdf/chessaton_gazebo.xacro (robot description, xacro)
@@ -64,4 +64,21 @@
         <implicitSpringDamper>1</implicitSpringDamper>
     </gazebo> -->
+    <gazebo>
+        <plugin name="gazebo_grasp_fix" filename="libgazebo_grasp_fix.so">
+             <arm>
+                <arm_name>chessaton</arm_name>
+                <palm_link> chessaton_link4  </palm_link>
+                <gripper_link> right_finger </gripper_link>
+                <gripper_link> left_finger </gripper_link>
+             </arm>
+            <forces_angle_tolerance>100</forces_angle_tolerance>
+            <update_rate>10</update_rate>
+            <grip_count_threshold>5</grip_count_threshold>
+            <max_grip_count>10</max_grip_count>
+            <release_tolerance>0.005</release_tolerance>
+            <disable_collisions_on_attach>false</disable_collisions_on_attach>
+            <contact_topic>__default_topic__</contact_topic>
+         </plugin>
+    </gazebo>
     <!--       -->
     <!-- Macro -->

Commit message: Modify: reduced the speed and velocity of gripper fingers

File: chessaton_description/urdf/chessaton.urdf (robot description, URDF)
Before this commit: robot chessaton, 12 links, 11 joints
Joints:
- joint left_finger_joint: limit lower=0 upper=0.03 effort=100 velocity=0.2 -> lower=0 upper=0.03 effort=100 velocity=0.02
- joint right_finger_joint: limit lower=-0.03 upper=0 effort=100 velocity=0.2 -> lower=-0.03 upper=0 effort=100 velocity=0.02

File: chessaton_description/urdf/chessaton_gazebo.xacro (robot description, xacro)
@@ -72,9 +72,9 @@
                 <gripper_link> left_finger </gripper_link>
              </arm>
-            <forces_angle_tolerance>100</forces_angle_tolerance>
-            <update_rate>10</update_rate>
+            <forces_angle_tolerance>120</forces_angle_tolerance>
+            <update_rate>30</update_rate>
             <grip_count_threshold>5</grip_count_threshold>
-            <max_grip_count>10</max_grip_count>
-            <release_tolerance>0.005</release_tolerance>
+            <max_grip_count>20</max_grip_count>
+            <release_tolerance>0.008</release_tolerance>
             <disable_collisions_on_attach>false</disable_collisions_on_attach>
             <contact_topic>__default_topic__</contact_topic>

File: chessaton_description/urdf/chessaton_hand.xacro (robot description, xacro)
@@ -40,5 +40,5 @@
     		<axis xyz="0 1 0" />
     		<dynamics damping="1.0" friction="1.0" />
-    		<limit lower="0" upper="0.03" effort="100" velocity="0.2" />
+    		<limit lower="0" upper="0.03" effort="100" velocity="0.02" />
     	</joint>
     	<link name="left_finger">
@@ -77,5 +77,5 @@
     		<axis xyz="0 1 0" />
     		<dynamics damping="1.0" friction="1.0" />
-    		<limit lower="-0.03" upper="0" effort="100" velocity="0.2" />
+    		<limit lower="-0.03" upper="0" effort="100" velocity="0.02" />
     	</joint>
     	<link name="right_finger">
