Commit message: Modify: changed the robot model (extended link 1 & 2)

File: chessaton_description/urdf/chessaton.urdf (robot description, URDF)
Before this commit: robot chessaton, 12 links, 11 joints
Links:
- link chessaton_link2: mass 0.045902162826317 -> 0.077067
- link chessaton_link3: mass 0.076498 -> 0.10766
- link chessaton_link4: mass 0.046643 -> 0.0466425419935174
Joints:
- joint chessaton_joint3: origin xyz=0 0 0.102 rpy=0 0 0 -> xyz=0 0 0.202 rpy=0 0 0
- joint chessaton_joint4: origin xyz=0.098504 0.00041731 0.0019578 rpy=0 0 0 -> xyz=0.1985 0.0019174 0.0019578 rpy=0 0 0

File: chessaton_description/urdf/chessaton.urdf.xacro (robot description, xacro)
@@ -116,13 +116,13 @@
         </visual>
         <inertial>
-            <origin xyz="1.94289029309402E-16 -0.0247721366408157 0.0510000000000001" rpy="0 0 0" />
-            <mass value="0.045902162826317" />
-            <inertia
-              ixx="4.65002565093796E-05"
-              ixy="2.26509482575262E-19"
-              ixz="1.10875380838109E-14"
-              iyy="2.11429163261091E-05"
-              iyz="-2.47808875423641E-23"
-              izz="3.01847862586687E-05" />
+            <origin xyz="1.1343E-09 -0.02475 0.101" rpy="0 0 0" />
+            <mass value="0.077067" />
+            <inertia
+              ixx="7.2952E-05"
+              ixy="4.5829E-12"
+              ixz="1.1087E-14"
+              iyy="4.7593E-05"
+              iyz="3.7988E-20"
+              izz="3.1748E-05" />
         </inertial>
         <collision>
@@ -134,5 +134,5 @@
     </link>
 	<joint name="chessaton_joint3" type="revolute">
-	  	<origin xyz="0 0 0.102" rpy="0 0 0" />
+	  	<origin xyz="0 0 0.202" rpy="0 0 0" />
 	  	<parent link="chessaton_link2" />
 	  	<child link="chessaton_link3" />
@@ -156,17 +156,17 @@
 		</collision>
 		<inertial>
-            <origin xyz="0.030212 -0.026096 -0.0011497" rpy="0 0 0" />
-            <mass value="0.076498" />
-            <inertia
-              ixx="2.3983E-05"
-              ixy="7.4374E-08"
+            <origin xyz="0.071008 -0.024827 -0.00025021" rpy="0 0 0" />
+            <mass value="0.10766" />
+            <inertia
+              ixx="2.5545E-05"
+              ixy="8.4872E-08"
               ixz="-3.21E-07"
-              iyy="2.2146E-05"
+              iyy="4.8596E-05"
               iyz="4.236E-07"
-              izz="3.9025E-05" />
+              izz="6.5475E-05" />
         </inertial>
 	</link>
 	<joint name="chessaton_joint4" type="revolute">
-	    <origin xyz="0.098504 0.00041731 0.0019578" rpy="0 0 0" />
+	    <origin xyz="0.1985 0.0019174 0.0019578" rpy="0 0 0" />
 	    <parent link="chessaton_link3" />
 	    <child link="chessaton_link4" />
@@ -191,8 +191,8 @@
         <inertial>
             <origin xyz="0.0016488 -0.027436 -0.0097099" rpy="0 0 0" />
-            <mass value="0.046643" />
+            <mass value="0.0466425419935174" />
             <inertia
               ixx="1.458E-05"
-              ixy="-4.236E-07"
+              ixy="-4.2359E-07"
               ixz="-1.6429E-09"
               iyy="1.0335E-05"

File: chessaton_description/urdf/chessaton_gazebo.xacro (robot description, xacro)
@@ -74,7 +74,7 @@
             <forces_angle_tolerance>120</forces_angle_tolerance>
             <update_rate>30</update_rate>
-            <grip_count_threshold>5</grip_count_threshold>
+            <grip_count_threshold>4</grip_count_threshold>
             <max_grip_count>20</max_grip_count>
-            <release_tolerance>0.008</release_tolerance>
+            <release_tolerance>0.002</release_tolerance>
             <disable_collisions_on_attach>false</disable_collisions_on_attach>
             <contact_topic>__default_topic__</contact_topic>

File: chessaton_description/urdf/chessaton_hand.xacro (robot description, xacro)
@@ -106,4 +106,12 @@
     	</link>
         <xacro:if value="${virtual_dof}">
+            <joint name="chessaton_hand_tcp_roll_virtual_joint" type="revolute">
+                <parent link="chessaton_gripper"/>
+                <child link="chessaton_hand_tcp_roll"/>
+                <origin rpy="0 0 0" xyz="0.02 0 -0.005"/>
+                <axis xyz="-1 0 0" />
+    		    <dynamics damping="1.0" friction="1.0" />
+    	        <limit lower="${-pi/2}" upper="${pi/2}" effort="0" velocity="6" />
+            </joint>
             <link name="chessaton_hand_tcp_roll">
                 <inertial>
@@ -119,12 +127,4 @@
                 </inertial>
             </link>
-            <joint name="chessaton_hand_tcp_roll_virtual_joint" type="revolute">
-                <parent link="chessaton_gripper"/>
-                <child link="chessaton_hand_tcp_roll"/>
-                <origin rpy="0 0 0" xyz="0.02 0 -0.005"/>
-                <axis xyz="-1 0 0" />
-    		<dynamics damping="1.0" friction="1.0" />
-    	     <limit lower="${-pi/2}" upper="${pi/2}" effort="0" velocity="6" />
-            </joint>
             <link name="chessaton_hand_tcp_yaw">
                 <inertial>

Commit message: Modify: changed design of gripper and base link.

File: chessaton_description/urdf/chessaton.urdf (robot description, URDF)
Before this commit: robot chessaton, 12 links, 11 joints
Links:
- link chessaton_link0: mass 0.094842 -> 0.17447
- link chessaton_link1: mass 0.047535 -> 0.046511
- link chessaton_link2: mass 0.077067 -> 0.070955
- link chessaton_link3: mass 0.10766 -> 0.099802
- link left_finger: mass 0.0088 -> 0.00601945436907758
- link right_finger: mass 0.0088 -> 0.0060194543690775
Joints:
- joint chessaton_hand_tcp_roll_virtual_joint: origin xyz=0.02 0 -0.005 rpy=0 0 0 -> xyz=0.03 0 0 rpy=0 0 0
- joint chessaton_joint1: limit lower=-3.141592653589793 upper=3.141592653589793 effort=0 velocity=5 -> lower=-1.5707963267948966 upper=1.5707963267948966 effort=0 velocity=5; origin xyz=0.00015368 0.01229 0.07705 rpy=0 0 0 -> xyz=0 0 0.08094 rpy=0 0 0
- joint chessaton_joint2: origin xyz=0.022504 0.022833 0.013792 rpy=0 0 0 -> xyz=0.022104 0.022723 0.015309 rpy=0 0 0
- joint chessaton_joint3: origin xyz=0 0 0.202 rpy=0 0 0 -> xyz=0 0 0.18701 rpy=0 0 0
- joint chessaton_joint4: origin xyz=0.1985 0.0019174 0.0019578 rpy=0 0 0 -> xyz=0.17811 0.0028273 9.1141E-05 rpy=0 0 0
- joint gripper_joint: origin xyz=0.072842 -0.034194 -0.0048547 rpy=0 0 0 -> xyz=0.070609 -0.033634 -0.0087075 rpy=0 0 0
- joint left_finger_joint: limit lower=0 upper=0.03 effort=100 velocity=0.02 -> lower=0 upper=0.023 effort=100 velocity=0.02
- joint right_finger_joint: limit lower=-0.03 upper=0 effort=100 velocity=0.02 -> lower=-0.023 upper=0 effort=100 velocity=0.02

File: chessaton_description/urdf/chessaton.urdf.xacro (robot description, xacro)
@@ -54,22 +54,22 @@
         </collision>
         <inertial>
-            <origin xyz="-0.00073528 0.0040282 0.031188" rpy="0 0 0" />
-            <mass value="0.094842" />
-            <inertia
-              ixx="3.0463E-05"
-              ixy="-6.3087E-09"
-              ixz="4.236E-07"
-              iyy="4.8143E-05"
-              iyz="-8.1925E-08"
-              izz="5.1511E-05" />
+            <origin xyz="-0.050129 -0.010271 0.035819" rpy="0 0 0" />
+            <mass value="0.17447" />
+            <inertia
+                ixx="0.00011969"
+                ixy="1.6753E-09"
+                ixz="4.5328E-07"
+                iyy="0.00034675"
+                iyz="-4.0946E-09"
+                izz="0.00045331" />
         </inertial>
     </link>
     <joint name="chessaton_joint1" type="revolute">
-        <origin xyz="0.00015368 0.01229 0.07705" rpy="0 0 0" />
+        <origin xyz="0 0 0.08094" rpy="0 0 0" />
         <parent link="chessaton_link0" />
         <child link="chessaton_link1" />
         <axis xyz="0 0 -1" />
 		<dynamics damping="1.0" friction="1.0" />
-        <limit lower="${-pi}" upper="${pi}" effort="0" velocity="5" />
+        <limit lower="${-pi/2}" upper="${pi/2}" effort="0" velocity="5" />
     </joint>
     <link name="chessaton_link1">
@@ -88,17 +88,17 @@
         </collision>
         <inertial>
-            <origin xyz="0.012256 -0.0045169 0.011915" rpy="0 0 0" />
-            <mass value="0.047535" />
-            <inertia
-              ixx="8.1555E-06"
-              ixy="-8.4986E-08"
-              ixz="1.6429E-09"
-              iyy="1.0365E-05"
-              iyz="4.236E-07"
-              izz="1.4637E-05" />
+            <origin xyz="0.012052 -0.0041948 0.012838" rpy="0 0 0" />
+            <mass value="0.046511" />
+            <inertia
+              ixx="7.7123E-06"
+              ixy="-4.0766E-09"
+              ixz="1.6732E-09"
+              iyy="1.046E-05"
+              iyz="4.5327E-07"
+              izz="1.4407E-05" />
         </inertial>
     </link>
 	<joint name="chessaton_joint2" type="revolute">
-		<origin xyz="0.022504 0.022833 0.013792" rpy="0 0 0" />
+		<origin xyz="0.022104 0.022723 0.015309" rpy="0 0 0" />
 		<parent link="chessaton_link1" />
 		<child link="chessaton_link2" />
@@ -116,13 +116,13 @@
         </visual>
         <inertial>
-            <origin xyz="1.1343E-09 -0.02475 0.101" rpy="0 0 0" />
-            <mass value="0.077067" />
-            <inertia
-              ixx="7.2952E-05"
-              ixy="4.5829E-12"
-              ixz="1.1087E-14"
-              iyy="4.7593E-05"
-              iyz="3.7988E-20"
-              izz="3.1748E-05" />
+            <origin xyz="-6.8198E-09 -0.0253 0.093503" rpy="0 0 0" />
+            <mass value="0.070955" />
+            <inertia
+              ixx="6.1321E-05"
+              ixy="7.7897E-20"
+              ixz="4.4464E-12"
+              iyy="3.639E-05"
+              iyz="-5.6971E-19"
+              izz="3.1036E-05" />
         </inertial>
         <collision>
@@ -134,5 +134,5 @@
     </link>
 	<joint name="chessaton_joint3" type="revolute">
-	  	<origin xyz="0 0 0.202" rpy="0 0 0" />
+	  	<origin xyz="0 0 0.18701" rpy="0 0 0" />
 	  	<parent link="chessaton_link2" />
 	  	<child link="chessaton_link3" />
@@ -156,17 +156,17 @@
 		</collision>
 		<inertial>
-            <origin xyz="0.071008 -0.024827 -0.00025021" rpy="0 0 0" />
-            <mass value="0.10766" />
-            <inertia
-              ixx="2.5545E-05"
-              ixy="8.4872E-08"
-              ixz="-3.21E-07"
-              iyy="4.8596E-05"
-              iyz="4.236E-07"
-              izz="6.5475E-05" />
+            <origin xyz="0.061953 -0.024546 -0.0017072" rpy="0 0 0" />
+            <mass value="0.099802" />
+            <inertia
+              ixx="2.455E-05"
+              ixy="6.6798E-10"
+              ixz="-2.7683E-07"
+              iyy="3.4978E-05"
+              iyz="4.5265E-07"
+              izz="5.1335E-05" />
         </inertial>
 	</link>
 	<joint name="chessaton_joint4" type="revolute">
-	    <origin xyz="0.1985 0.0019174 0.0019578" rpy="0 0 0" />
+	    <origin xyz="0.17811 0.0028273 9.1141E-05" rpy="0 0 0" />
 	    <parent link="chessaton_link3" />
 	    <child link="chessaton_link4" />
@@ -190,17 +190,17 @@
 		</collision>
         <inertial>
-            <origin xyz="0.0016488 -0.027436 -0.0097099" rpy="0 0 0" />
+            <origin xyz="0.00247132842176606 -0.0269174421054227 -0.0100525933944812" rpy="0 0 0" />
             <mass value="0.0466425419935174" />
             <inertia
-              ixx="1.458E-05"
-              ixy="-4.2359E-07"
-              ixz="-1.6429E-09"
-              iyy="1.0335E-05"
-              iyz="-8.4986E-08"
-              izz="8.1259E-06" />
+              ixx="1.4406877106279E-05"
+              ixy="-4.53266983583288E-07"
+              ixz="-1.6729067017079E-09"
+              iyy="1.04604416782095E-05"
+              iyz="-4.07637977779482E-09"
+              izz="7.71225534218515E-06" />
         </inertial>
 	</link>
 	<joint name="gripper_joint" type="fixed">
-	  <origin xyz="0.072842 -0.034194 -0.0048547" rpy="0 0 0" />
+	  <origin xyz="0.070609 -0.033634 -0.0087075" rpy="0 0 0" />
 	  <parent link="chessaton_link4" />
 	  <child link="chessaton_gripper" />

File: chessaton_description/urdf/chessaton_hand.xacro (robot description, xacro)
@@ -23,13 +23,13 @@
     		</collision>
             <inertial>
-                <origin xyz="-0.027242 0.0063062 -0.003963" rpy="0 0 0" />
+                <origin xyz="-0.0266113093832042 -0.00792294858682179 -0.00177094549286488" rpy="0 0 0" />
                 <mass value="0.07416" />
                 <inertia
-                  ixx="2.5968E-05"
-                  ixy="8.488E-08"
-                  ixz="-4.236E-07"
-                  iyy="1.3082E-05"
-                  iyz="-1.6429E-09"
-                  izz="2.6136E-05" />
+                  ixx="1.94087256012664E-05"
+                  ixy="-4.11947485817516E-09"
+                  ixz="4.53529646177736E-07"
+                  iyy="9.16253998980345E-06"
+                  iyz="-1.67298780752208E-09"
+                  izz="2.20817956679352E-05" />
             </inertial>
     	</link>
@@ -40,5 +40,5 @@
     		<axis xyz="0 1 0" />
     		<dynamics damping="1.0" friction="1.0" />
-    		<limit lower="0" upper="0.03" effort="100" velocity="0.02" />
+    		<limit lower="0" upper="0.023" effort="100" velocity="0.02" />
     	</joint>
     	<link name="left_finger">
@@ -58,15 +58,15 @@
             <inertial>
                 <origin
-                  xyz="0.011394 0.0086324 -0.005"
+                  xyz="0.0127036998303536 0.00249799647668462 0.00302307598216517"
                   rpy="0 0 0" />
                 <mass
-                  value="0.0088" />
+                  value="0.00601945436907758" />
                 <inertia
-                  ixx="6.0646E-07"
-                  ixy="1.4141E-07"
-                  ixz="2.4551E-21"
-                  iyy="9.0397E-07"
-                  iyz="-6.5992E-22"
-                  izz="8.4377E-07" />
+                  ixx="8.35687237301018E-07"
+                  ixy="-1.33370717821302E-07"
+                  ixz="1.71869210411339E-07"
+                  iyy="1.12520988095806E-06"
+                  iyz="1.94902986855749E-07"
+                  izz="1.56286387867122E-06" />
             </inertial>
     	</link>
@@ -77,5 +77,5 @@
     		<axis xyz="0 1 0" />
     		<dynamics damping="1.0" friction="1.0" />
-    		<limit lower="-0.03" upper="0" effort="100" velocity="0.02" />
+    		<limit lower="-0.023" upper="0" effort="100" velocity="0.02" />
     	</joint>
     	<link name="right_finger">
@@ -94,13 +94,13 @@
     		</collision>
             <inertial>
-                <origin xyz="0.011394 -0.0086324 -0.005" rpy="0 0 0" />
-                <mass value="0.0088" />
+                <origin xyz="0.0127036998303538 -0.00154590959997161 -0.00302307586801204" rpy="0 0 0" />
+                <mass value="0.0060194543690775" />
                 <inertia
-                  ixx="6.0646E-07"
-                  ixy="-1.4141E-07"
-                  ixz="1.2142E-21"
-                  iyy="9.0397E-07"
-                  iyz="7.2151E-22"
-                  izz="8.4377E-07" />
+                  ixx="8.35687237301015E-07"
+                  ixy="1.33370717821309E-07"
+                  ixz="-1.71869210411314E-07"
+                  iyy="1.12520988095806E-06"
+                  iyz="1.94902986855771E-07"
+                  izz="1.5628638786712E-06" />
             </inertial>
     	</link>
@@ -109,5 +109,5 @@
                 <parent link="chessaton_gripper"/>
                 <child link="chessaton_hand_tcp_roll"/>
-                <origin rpy="0 0 0" xyz="0.02 0 -0.005"/>
+                <origin rpy="0 0 0" xyz="0.03 0 0"/>
                 <axis xyz="-1 0 0" />
     		    <dynamics damping="1.0" friction="1.0" />
@@ -162,5 +162,5 @@
               <parent link="chessaton_gripper"/>
               <child link="chessaton_hand_tcp"/>
-              <origin rpy="0 0 0" xyz="0.02 0 -0.005"/>
+              <origin rpy="0 0 0" xyz="0.03 0 0"/>
             </joint>
         </xacro:unless>

File: chessaton_moveit_config/srdf/chessaton_macro.srdf.xacro (robot description, xacro)
@@ -39,6 +39,6 @@
         </group_state>
         <group_state name="hand_open" group="chessaton_hand">
-            <joint name="left_finger_joint" value="0.03"/>
-            <joint name="right_finger_joint" value="-0.03"/>
+            <joint name="left_finger_joint" value="0.023"/>
+            <joint name="right_finger_joint" value="-0.023"/>
         </group_state>
         <group name="chessaton_arm_hand">

Commit message: Fix: fixed gripper gap and gazebo angle tolerance

File: chessaton_description/urdf/chessaton.urdf (robot description, URDF)
Before this commit: robot chessaton, 12 links, 11 joints
Links:
- link chessaton_gripper: mass 0.07416 -> 0.06585

File: chessaton_description/urdf/chessaton.urdf.xacro (robot description, xacro)
@@ -1,3 +1,3 @@
-<?xml version="0.5" encoding="utf-8"?>
+<?xml version="1.0" encoding="utf-8"?>
 <robot xmlns:xacro="http://www.ros.org/wiki/xacro"
     xmlns:sensor="http://playerstage.sourceforge.net/gazebo/xmlschema/#sensor"

File: chessaton_description/urdf/chessaton_gazebo.xacro (robot description, xacro)
@@ -72,5 +72,5 @@
                 <gripper_link> left_finger </gripper_link>
              </arm>
-            <forces_angle_tolerance>120</forces_angle_tolerance>
+            <forces_angle_tolerance>140</forces_angle_tolerance>
             <update_rate>30</update_rate>
             <grip_count_threshold>4</grip_count_threshold>

File: chessaton_description/urdf/chessaton_hand.xacro (robot description, xacro)
@@ -23,6 +23,6 @@
     		</collision>
             <inertial>
-                <origin xyz="-0.0266113093832042 -0.00792294858682179 -0.00177094549286488" rpy="0 0 0" />
-                <mass value="0.07416" />
+                <origin xyz="-0.0266113093832023 -0.00796252580865704 -0.00177094549286499" rpy="0 0 0" />
+                <mass value="0.06585" />
                 <inertia
                   ixx="1.94087256012664E-05"
@@ -58,13 +58,13 @@
             <inertial>
                 <origin
-                  xyz="0.0127036998303536 0.00249799647668462 0.00302307598216517"
+                  xyz="0.0127036998303557 0.00154590778352602 0.00302307598216484"
                   rpy="0 0 0" />
                 <mass
                   value="0.00601945436907758" />
                 <inertia
-                  ixx="8.35687237301018E-07"
-                  ixy="-1.33370717821302E-07"
+                  ixx="8.35687237301017E-07"
+                  ixy="-1.33370717821303E-07"
                   ixz="1.71869210411339E-07"
-                  iyy="1.12520988095806E-06"
+                  iyy="1.12520988095805E-06"
                   iyz="1.94902986855749E-07"
                   izz="1.56286387867122E-06" />
@@ -94,12 +94,12 @@
     		</collision>
             <inertial>
-                <origin xyz="0.0127036998303538 -0.00154590959997161 -0.00302307586801204" rpy="0 0 0" />
+                <origin xyz="0.0127036998303559 -0.00154590852707946 -0.00302307586801259" rpy="0 0 0" />
                 <mass value="0.0060194543690775" />
                 <inertia
-                  ixx="8.35687237301015E-07"
-                  ixy="1.33370717821309E-07"
-                  ixz="-1.71869210411314E-07"
+                  ixx="8.35687237301014E-07"
+                  ixy="1.33370717821308E-07"
+                  ixz="-1.71869210411315E-07"
                   iyy="1.12520988095806E-06"
-                  iyz="1.94902986855771E-07"
+                  iyz="1.9490298685577E-07"
                   izz="1.5628638786712E-06" />
             </inertial>
