Commit message: Modify: change in design, add rotary plate and an extra motor to second link

File: chessaton_description/urdf/chessaton.urdf (robot description, URDF)
Before this commit: robot chessaton, 12 links, 11 joints
Links:
- link chessaton_hand_tcp: mass None -> 0.0088
- link chessaton_link0: mass 0.17447 -> 0.35099
- link chessaton_link1: mass 0.046511 -> 0.11596191407717
- link chessaton_link3: mass 0.099802 -> 0.01
- link chessaton_link4: mass 0.0466425419935174 -> 0.0465
- link left_finger: mass 0.00601945436907758 -> 0.006
- link right_finger: mass 0.0060194543690775 -> 0.006
Joints:
- joint chessaton_joint1: limit lower=-1.5707963267948966 upper=1.5707963267948966 effort=0 velocity=5 -> lower=-1.5707963267948966 upper=1.5707963267948966 effort=0 velocity=0.2618; origin xyz=0 0 0.08094 rpy=0 0 0 -> xyz=0 0 0.07184 rpy=0 0 0
- joint chessaton_joint2: axis 0 -1 0 -> 0 1 0; limit lower=-1.5707963267948966 upper=1.5707963267948966 effort=0 velocity=5 -> lower=-1.5707963267948966 upper=1.5707963267948966 effort=0 velocity=0.2618; origin xyz=0.022104 0.022723 0.015309 rpy=0 0 0 -> xyz=0 1.2977E-05 0.030569 rpy=0 0 0
- joint chessaton_joint3: axis 0 -1 0 -> 0 1 0; limit lower=-1.5707963267948966 upper=1.5707963267948966 effort=0 velocity=6 -> lower=-1.5707963267948966 upper=1.5707963267948966 effort=0 velocity=0.2618; origin xyz=0 0 0.18701 rpy=0 0 0 -> xyz=0 0.025346 0.18701 rpy=0 0 0
- joint chessaton_joint4: axis 0 -1 0 -> 0 1 0; limit lower=-1.5707963267948966 upper=1.5707963267948966 effort=0 velocity=6 -> lower=-1.5707963267948966 upper=1.5707963267948966 effort=0 velocity=0.2618; origin xyz=0.17811 0.0028273 9.1141E-05 rpy=0 0 0 -> xyz=0.17811 0.0028223 9.1137E-05 rpy=0 0 0
- joint gripper_joint: origin xyz=0.070609 -0.033634 -0.0087075 rpy=0 0 0 -> xyz=0.070608 -0.033636 -0.0087075 rpy=0 0 0
- joint left_finger_joint: limit lower=0 upper=0.023 effort=100 velocity=0.02 -> lower=0 upper=0.023 effort=100 velocity=0.01
- joint right_finger_joint: limit lower=-0.023 upper=0 effort=100 velocity=0.02 -> lower=-0.023 upper=0 effort=100 velocity=0.01

File: chessaton_description/urdf/chessaton.urdf.xacro (robot description, xacro)
@@ -54,22 +54,22 @@
         </collision>
         <inertial>
-            <origin xyz="-0.050129 -0.010271 0.035819" rpy="0 0 0" />
-            <mass value="0.17447" />
-            <inertia
-                ixx="0.00011969"
-                ixy="1.6753E-09"
-                ixz="4.5328E-07"
-                iyy="0.00034675"
-                iyz="-4.0946E-09"
-                izz="0.00045331" />
+            <origin xyz="-0.00088323 -3.593E-07 0.021799" rpy="0 0 0" />
+            <mass value="0.35099" />
+            <inertia
+                ixx="0.00040857"
+                ixy="-1.2568E-09"
+                ixz="-4.0915E-09"
+                iyy="0.00041214"
+                iyz="1.5948E-10"
+                izz="0.00079973" />
         </inertial>
     </link>
     <joint name="chessaton_joint1" type="revolute">
-        <origin xyz="0 0 0.08094" rpy="0 0 0" />
+        <origin xyz="0 0 0.07184" rpy="0 0 0" />
         <parent link="chessaton_link0" />
         <child link="chessaton_link1" />
         <axis xyz="0 0 -1" />
-		<dynamics damping="0.5" friction="0.0" />
-        <limit lower="${-pi/2}" upper="${pi/2}" effort="0" velocity="5" />
+		<dynamics damping="0.01" friction="0.01" />
+        <limit lower="${-pi/2}" upper="${pi/2}" effort="0" velocity="0.2618" />
     </joint>
     <link name="chessaton_link1">
@@ -88,22 +88,22 @@
         </collision>
         <inertial>
-            <origin xyz="0.012052 -0.0041948 0.012838" rpy="0 0 0" />
-            <mass value="0.046511" />
-            <inertia
-              ixx="7.7123E-06"
-              ixy="-4.0766E-09"
-              ixz="1.6732E-09"
-              iyy="1.046E-05"
-              iyz="4.5327E-07"
-              izz="1.4407E-05" />
+            <origin xyz="-2.48292998257112E-06 1.80948923297683E-11 0.0255783185959284" rpy="0 0 0" />
+            <mass value="0.11596191407717" />
+            <inertia
+              ixx="5.46629273225896E-05"
+              ixy="-1.33156669187786E-07"
+              ixz="3.35258624200402E-14"
+              iyy="4.25165415022482E-05"
+              iyz="-8.2983289116076E-14"
+              izz="8.94434749602387E-05" />
         </inertial>
     </link>
 	<joint name="chessaton_joint2" type="revolute">
-		<origin xyz="0.022104 0.022723 0.015309" rpy="0 0 0" />
+		<origin xyz="0 1.2977E-05 0.030569" rpy="0 0 0" />
 		<parent link="chessaton_link1" />
 		<child link="chessaton_link2" />
-		<axis xyz="0 -1 0" />
-		<dynamics damping="0.5" friction="0.0" />
-		<limit lower="${-pi/2}" upper="${pi/2}" effort="0" velocity="5" />
+		<axis xyz="0 1 0" />
+		<dynamics damping="0.01" friction="0.01" />
+		<limit lower="${-pi/2}" upper="${pi/2}" effort="0" velocity="0.2618" />
 	</joint>
     <link name="chessaton_link2">
@@ -116,12 +116,12 @@
         </visual>
         <inertial>
-            <origin xyz="-6.8198E-09 -0.0253 0.093503" rpy="0 0 0" />
+            <origin xyz="-2.3338E-06 4.5723E-05 0.093503" rpy="0 0 0" />
             <mass value="0.070955" />
             <inertia
               ixx="6.1321E-05"
-              ixy="7.7897E-20"
-              ixz="4.4464E-12"
+              ixy="-6.9447E-10"
+              ixz="4.4166E-12"
               iyy="3.639E-05"
-              iyz="-5.6971E-19"
+              iyz="-4.4751E-13"
               izz="3.1036E-05" />
         </inertial>
@@ -134,10 +134,10 @@
     </link>
 	<joint name="chessaton_joint3" type="revolute">
-	  	<origin xyz="0 0 0.18701" rpy="0 0 0" />
+	  	<origin xyz="0 0.025346 0.18701" rpy="0 0 0" />
 	  	<parent link="chessaton_link2" />
 	  	<child link="chessaton_link3" />
-	  	<axis xyz="0 -1 0" />
-	  	<dynamics damping="0.5" friction="0.0" />
-	  	<limit lower="${-pi/2}" upper="${pi/2}" effort="0" velocity="6" />
+	  	<axis xyz="0 1 0" />
+	  	<dynamics damping="0.01" friction="0.01" />
+	  	<limit lower="${-pi/2}" upper="${pi/2}" effort="0" velocity="0.2618" />
 	</joint>
 	<link name="chessaton_link3">
@@ -156,22 +156,22 @@
 		</collision>
 		<inertial>
-            <origin xyz="0.061953 -0.024546 -0.0017072" rpy="0 0 0" />
-            <mass value="0.099802" />
-            <inertia
-              ixx="2.455E-05"
-              ixy="6.6798E-10"
-              ixz="-2.7683E-07"
-              iyy="3.4978E-05"
-              iyz="4.5265E-07"
-              izz="5.1335E-05" />
+            <origin xyz="0.0619519890876748 -0.0245474768443102 -0.00170721074679331" rpy="0 0 0" />
+            <mass value="0.01" />
+            <inertia
+              ixx="2.45504457142139E-05"
+              ixy="9.48952036737489E-10"
+              ixz="-2.76965747257156E-07"
+              iyy="3.49778436797956E-05"
+              iyz="4.52657683759416E-07"
+              izz="5.13350744770814E-05" />
         </inertial>
 	</link>
 	<joint name="chessaton_joint4" type="revolute">
-	    <origin xyz="0.17811 0.0028273 9.1141E-05" rpy="0 0 0" />
+	    <origin xyz="0.17811 0.0028223 9.1137E-05" rpy="0 0 0" />
 	    <parent link="chessaton_link3" />
 	    <child link="chessaton_link4" />
-	    <axis xyz="0 -1 0" />
-		<dynamics damping="0.5" friction="0.0" />
-	    <limit lower="${-pi/2}" upper="${pi/2}" effort="0" velocity="6" />
+	    <axis xyz="0 1 0" />
+		<dynamics damping="0.01" friction="0.01" />
+	    <limit lower="${-pi/2}" upper="${pi/2}" effort="0" velocity="0.2618" />
 	</joint>
 	<link name="chessaton_link4">
@@ -190,17 +190,17 @@
 		</collision>
         <inertial>
-            <origin xyz="0.00247132842176606 -0.0269174421054227 -0.0100525933944812" rpy="0 0 0" />
-            <mass value="0.0466425419935174" />
-            <inertia
-              ixx="1.4406877106279E-05"
-              ixy="-4.53266983583288E-07"
-              ixz="-1.6729067017079E-09"
-              iyy="1.04604416782095E-05"
-              iyz="-4.07637977779482E-09"
-              izz="7.71225534218515E-06" />
+            <origin xyz="0.00247057855143362 -0.0269175108707789 -0.0100531530882181" rpy="0 0 0" />
+            <mass value="0.0465" />
+            <inertia
+              ixx="1.44068897410675E-05"
+              ixy="-4.53376917177043E-07"
+              ixz="-1.53060923766455E-09"
+              iyy="1.04605048186758E-05"
+              iyz="-4.07815450494968E-09"
+              izz="7.71225538228526E-06" />
         </inertial>
 	</link>
 	<joint name="gripper_joint" type="fixed">
-	  <origin xyz="0.070609 -0.033634 -0.0087075" rpy="0 0 0" />
+	  <origin xyz="0.070608 -0.033636 -0.0087075" rpy="0 0 0" />
 	  <parent link="chessaton_link4" />
 	  <child link="chessaton_gripper" />

File: chessaton_description/urdf/chessaton_hand.xacro (robot description, xacro)
@@ -23,13 +23,13 @@
     		</collision>
             <inertial>
-                <origin xyz="-0.0266113093832023 -0.00796252580865704 -0.00177094549286499" rpy="0 0 0" />
+                <origin xyz="-0.0266115313266715 -0.00796138911947138 -0.00177094547635764" rpy="0 0 0" />
                 <mass value="0.06585" />
                 <inertia
-                  ixx="1.94087256012664E-05"
-                  ixy="-4.11947485817516E-09"
-                  ixz="4.53529646177736E-07"
-                  iyy="9.16253998980345E-06"
-                  iyz="-1.67298780752208E-09"
-                  izz="2.20817956679352E-05" />
+                  ixx="1.94087633896407E-05"
+                  ixy="-4.40301296709736E-09"
+                  ixz="4.53529613378857E-07"
+                  iyy="9.16254031981619E-06"
+                  iyz="-1.54322487670811E-09"
+                  izz="2.20818336953172E-05" />
             </inertial>
     	</link>
@@ -40,5 +40,5 @@
     		<axis xyz="0 1 0" />
     		<dynamics damping="1.0" friction="1.0" />
-    		<limit lower="0" upper="0.023" effort="100" velocity="0.02" />
+    		<limit lower="0" upper="0.023" effort="100" velocity="0.01" />
     	</joint>
     	<link name="left_finger">
@@ -58,15 +58,15 @@
             <inertial>
                 <origin
-                  xyz="0.0127036998303557 0.00154590778352602 0.00302307598216484"
+                  xyz="0.0127034645973708 0.00154565127207735 0.0030231093837057"
                   rpy="0 0 0" />
                 <mass
-                  value="0.00601945436907758" />
+                  value="0.006" />
                 <inertia
-                  ixx="8.35687237301017E-07"
-                  ixy="-1.33370717821303E-07"
-                  ixz="1.71869210411339E-07"
-                  iyy="1.12520988095805E-06"
-                  iyz="1.94902986855749E-07"
-                  izz="1.56286387867122E-06" />
+                  ixx="8.35673086475568E-07"
+                  ixy="-1.33373055978949E-07"
+                  ixz="1.71871382347731E-07"
+                  iyy="1.12518172710191E-06"
+                  iyz="1.94898487683555E-07"
+                  izz="1.56282552281173E-06" />
             </inertial>
     	</link>
@@ -77,5 +77,5 @@
     		<axis xyz="0 1 0" />
     		<dynamics damping="1.0" friction="1.0" />
-    		<limit lower="-0.023" upper="0" effort="100" velocity="0.02" />
+    		<limit lower="-0.023" upper="0" effort="100" velocity="0.01" />
     	</joint>
     	<link name="right_finger">
@@ -94,13 +94,13 @@
     		</collision>
             <inertial>
-                <origin xyz="0.0127036998303559 -0.00154590852707946 -0.00302307586801259" rpy="0 0 0" />
-                <mass value="0.0060194543690775" />
+                <origin xyz="0.0127037648728564 -0.00154618659083175 -0.00302306815560061" rpy="0 0 0" />
+                <mass value="0.006" />
                 <inertia
-                  ixx="8.35687237301014E-07"
-                  ixy="1.33370717821308E-07"
-                  ixz="-1.71869210411315E-07"
-                  iyy="1.12520988095806E-06"
-                  iyz="1.9490298685577E-07"
-                  izz="1.5628638786712E-06" />
+                  ixx="8.35698479109993E-07"
+                  ixy="1.33368292398724E-07"
+                  ixz="-1.71864622126188E-07"
+                  iyy="1.1252213355056E-06"
+                  iyz="1.94907513457399E-07"
+                  izz="1.56288435175142E-06" />
             </inertial>
     	</link>
@@ -149,4 +149,15 @@
             </joint>
             <link name="chessaton_hand_tcp">
+                <inertial>
+                    <origin xyz="0.011394 -0.0086324 -0.005" rpy="0 0 0" />
+                    <mass value="0.0088" />
+                    <inertia
+                      ixx="6.0646E-07"
+                      ixy="-1.4141E-07"
+                      ixz="1.2142E-21"
+                      iyy="9.0397E-07"
+                      iyz="7.2151E-22"
+                      izz="8.4377E-07" />
+                </inertial>
             </link>
             <joint name="chessaton_hand_tcp_virtual_joint" type="fixed">
@@ -158,4 +169,15 @@
         <xacro:unless value="${virtual_dof}">
             <link name="chessaton_hand_tcp">
+                <inertial>
+                    <origin xyz="0.011394 -0.0086324 -0.005" rpy="0 0 0" />
+                    <mass value="0.0088" />
+                    <inertia
+                      ixx="6.0646E-07"
+                      ixy="-1.4141E-07"
+                      ixz="1.2142E-21"
+                      iyy="9.0397E-07"
+                      iyz="7.2151E-22"
+                      izz="8.4377E-07" />
+                </inertial>
             </link>
             <joint name="chessaton_hand_tcp_virtual_joint" type="fixed">
