Commit message: Modify: slight modification in design and adjusting the speed of joints.

File: chessaton_description/urdf/chessaton.urdf (robot description, URDF)
Before this commit: robot chessaton, 12 links, 11 joints
Links:
- link chessaton_gripper: mass 0.06585 -> 0.066
- link chessaton_link0: mass 0.35099 -> 0.35
- link chessaton_link1: mass 0.11596191407717 -> 0.116
- link chessaton_link2: mass 0.070955 -> 0.071
Joints:
- joint chessaton_joint1: limit lower=-1.5707963267948966 upper=1.5707963267948966 effort=0 velocity=0.2618 -> lower=-1.5707963267948966 upper=1.5707963267948966 effort=0 velocity=0.3
- joint chessaton_joint2: limit lower=-1.5707963267948966 upper=1.5707963267948966 effort=0 velocity=0.2618 -> lower=-1.5707963267948966 upper=1.5707963267948966 effort=0 velocity=0.3; origin xyz=0 1.2977E-05 0.030569 rpy=0 0 0 -> xyz=0 1.29770906784333E-05 0.0305688591051693 rpy=0 0 0
- joint chessaton_joint3: limit lower=-1.5707963267948966 upper=1.5707963267948966 effort=0 velocity=0.2618 -> lower=-1.5707963267948966 upper=1.5707963267948966 effort=0 velocity=0.3; origin xyz=0 0.025346 0.18701 rpy=0 0 0 -> xyz=0 0.025345720651074 0.187006906655083 rpy=0 0 0
- joint chessaton_joint4: limit lower=-1.5707963267948966 upper=1.5707963267948966 effort=0 velocity=0.2618 -> lower=-1.5707963267948966 upper=1.5707963267948966 effort=0 velocity=0.3; origin xyz=0.17811 0.0028223 9.1137E-05 rpy=0 0 0 -> xyz=0.157407990853242 0.00282292319687479 -0.000108863252950619 rpy=0 0 0
- joint gripper_joint: origin xyz=0.070608 -0.033636 -0.0087075 rpy=0 0 0 -> xyz=0.070608507146197 -0.0126359232516508 -0.0087074752469517 rpy=0 0 0

File: chessaton_description/urdf/chessaton.urdf.xacro (robot description, xacro)
@@ -55,5 +55,5 @@
         <inertial>
             <origin xyz="-0.00088323 -3.593E-07 0.021799" rpy="0 0 0" />
-            <mass value="0.35099" />
+            <mass value="0.35" />
             <inertia
                 ixx="0.00040857"
@@ -70,6 +70,6 @@
         <child link="chessaton_link1" />
         <axis xyz="0 0 -1" />
-		<dynamics damping="0.01" friction="0.01" />
-        <limit lower="${-pi/2}" upper="${pi/2}" effort="0" velocity="0.2618" />
+		<dynamics damping="0.1" friction="0.1" />
+        <limit lower="${-pi/2}" upper="${pi/2}" effort="0" velocity="0.3" />
     </joint>
     <link name="chessaton_link1">
@@ -88,22 +88,22 @@
         </collision>
         <inertial>
-            <origin xyz="-2.48292998257112E-06 1.80948923297683E-11 0.0255783185959284" rpy="0 0 0" />
-            <mass value="0.11596191407717" />
-            <inertia
-              ixx="5.46629273225896E-05"
-              ixy="-1.33156669187786E-07"
-              ixz="3.35258624200402E-14"
-              iyy="4.25165415022482E-05"
-              iyz="-8.2983289116076E-14"
-              izz="8.94434749602387E-05" />
+            <origin xyz="-2.4829E-06 1.8095E-11 0.025578" rpy="0 0 0" />
+            <mass value="0.116" />
+            <inertia
+              ixx="5.4663E-05"
+              ixy="-1.3316E-07"
+              ixz="3.3526E-14"
+              iyy="4.2517E-05"
+              iyz="-8.2983E-14"
+              izz="8.9443E-05" />
         </inertial>
     </link>
 	<joint name="chessaton_joint2" type="revolute">
-		<origin xyz="0 1.2977E-05 0.030569" rpy="0 0 0" />
+		<origin xyz="0 1.29770906784333E-05 0.0305688591051693" rpy="0 0 0" />
 		<parent link="chessaton_link1" />
 		<child link="chessaton_link2" />
 		<axis xyz="0 1 0" />
-		<dynamics damping="0.01" friction="0.01" />
-		<limit lower="${-pi/2}" upper="${pi/2}" effort="0" velocity="0.2618" />
+		<dynamics damping="0.1" friction="0.1" />
+		<limit lower="${-pi/2}" upper="${pi/2}" effort="0" velocity="0.3" />
 	</joint>
     <link name="chessaton_link2">
@@ -117,5 +117,5 @@
         <inertial>
             <origin xyz="-2.3338E-06 4.5723E-05 0.093503" rpy="0 0 0" />
-            <mass value="0.070955" />
+            <mass value="0.071" />
             <inertia
               ixx="6.1321E-05"
@@ -134,10 +134,10 @@
     </link>
 	<joint name="chessaton_joint3" type="revolute">
-	  	<origin xyz="0 0.025346 0.18701" rpy="0 0 0" />
+	  	<origin xyz="0 0.025345720651074 0.187006906655083" rpy="0 0 0" />
 	  	<parent link="chessaton_link2" />
 	  	<child link="chessaton_link3" />
 	  	<axis xyz="0 1 0" />
-	  	<dynamics damping="0.01" friction="0.01" />
-	  	<limit lower="${-pi/2}" upper="${pi/2}" effort="0" velocity="0.2618" />
+	  	<dynamics damping="0.1" friction="0.1" />
+	  	<limit lower="${-pi/2}" upper="${pi/2}" effort="0" velocity="0.3" />
 	</joint>
 	<link name="chessaton_link3">
@@ -156,22 +156,22 @@
 		</collision>
 		<inertial>
-            <origin xyz="0.0619519890876748 -0.0245474768443102 -0.00170721074679331" rpy="0 0 0" />
+            <origin xyz="0.041523 -0.024547 -0.0018439" rpy="0 0 0" />
             <mass value="0.01" />
             <inertia
-              ixx="2.45504457142139E-05"
-              ixy="9.48952036737489E-10"
-              ixz="-2.76965747257156E-07"
-              iyy="3.49778436797956E-05"
-              iyz="4.52657683759416E-07"
-              izz="5.13350744770814E-05" />
+              ixx="2.455E-05"
+              ixy="-7.247E-09"
+              ixz="-2.7697E-07"
+              iyy="3.4978E-05"
+              iyz="4.524E-07"
+              izz="5.1335E-05" />
         </inertial>
 	</link>
 	<joint name="chessaton_joint4" type="revolute">
-	    <origin xyz="0.17811 0.0028223 9.1137E-05" rpy="0 0 0" />
+	    <origin xyz="0.157407990853242 0.00282292319687479 -0.000108863252950619" rpy="0 0 0" />
 	    <parent link="chessaton_link3" />
 	    <child link="chessaton_link4" />
 	    <axis xyz="0 1 0" />
-		<dynamics damping="0.01" friction="0.01" />
-	    <limit lower="${-pi/2}" upper="${pi/2}" effort="0" velocity="0.2618" />
+		<dynamics damping="0.1" friction="0.1" />
+	    <limit lower="${-pi/2}" upper="${pi/2}" effort="0" velocity="0.3" />
 	</joint>
 	<link name="chessaton_link4">
@@ -190,17 +190,17 @@
 		</collision>
         <inertial>
-            <origin xyz="0.00247057855143362 -0.0269175108707789 -0.0100531530882181" rpy="0 0 0" />
+            <origin xyz="0.0024706 -0.026918 -0.010053" rpy="0 0 0" />
             <mass value="0.0465" />
             <inertia
-              ixx="1.44068897410675E-05"
-              ixy="-4.53376917177043E-07"
-              ixz="-1.53060923766455E-09"
-              iyy="1.04605048186758E-05"
-              iyz="-4.07815450494968E-09"
-              izz="7.71225538228526E-06" />
+              ixx="1.4407E-05"
+              ixy="-4.5338E-07"
+              ixz="-1.5306E-09"
+              iyy="1.0461E-05"
+              iyz="-4.0782E-09"
+              izz="7.7123E-06" />
         </inertial>
 	</link>
 	<joint name="gripper_joint" type="fixed">
-	  <origin xyz="0.070608 -0.033636 -0.0087075" rpy="0 0 0" />
+	  <origin xyz="0.070608507146197 -0.0126359232516508 -0.0087074752469517" rpy="0 0 0" />
 	  <parent link="chessaton_link4" />
 	  <child link="chessaton_gripper" />

File: chessaton_description/urdf/chessaton_gazebo.xacro (robot description, xacro)
@@ -8,5 +8,5 @@
         <kp value="1000000.0"/>
         <kd value="1.0"/>
-        <material>Gazebo/Green</material>
+    <material>Gazebo/Grey</material>
     </gazebo>
     <gazebo reference="chessaton_link1">
@@ -15,5 +15,5 @@
         <kp value="1000000.0"/>
         <kd value="1.0"/>
-        <material>Gazebo/Blue</material>
+        <material>Gazebo/Grey</material>
     </gazebo>
     <gazebo reference="chessaton_link2">
@@ -22,5 +22,5 @@
         <kp value="1000000.0"/>
         <kd value="1.0"/>
-        <material>Gazebo/Orange</material>
+        <material>Gazebo/Grey</material>
     </gazebo>
     <gazebo reference="chessaton_link3">
@@ -29,5 +29,5 @@
         <kp value="1000000.0"/>
         <kd value="1.0"/>
-        <material>Gazebo/Red</material>
+        <material>Gazebo/Grey</material>
     </gazebo>
     <gazebo reference="chessaton_link4">
@@ -36,5 +36,5 @@
         <kp value="1000000.0"/>
         <kd value="1.0"/>
-        <material>Gazebo/Black</material>
+        <material>Gazebo/Grey</material>
     </gazebo>
     <gazebo reference="chessaton_gripper">
@@ -43,5 +43,5 @@
         <kp value="1000000.0"/>
         <kd value="1.0"/>
-        <material>Gazebo/White</material>
+        <material>Gazebo/Grey</material>
     </gazebo>
     <gazebo reference="left_finger">
@@ -51,5 +51,5 @@
         <kd value="1.0"/>
         <minDepth>0.001</minDepth>
-        <material>Gazebo/White</material>
+        <material>Gazebo/Grey</material>
     </gazebo>
     <gazebo reference="right_finger">
@@ -59,5 +59,5 @@
         <kd value="1.0"/>
         <minDepth>0.001</minDepth>
-        <material>Gazebo/White</material>
+        <material>Gazebo/Grey</material>
     </gazebo>
     <!-- <gazebo reference="[joint name]">
@@ -72,9 +72,9 @@
                 <gripper_link> left_finger </gripper_link>
              </arm>
-            <forces_angle_tolerance>140</forces_angle_tolerance>
-            <update_rate>30</update_rate>
-            <grip_count_threshold>4</grip_count_threshold>
+            <forces_angle_tolerance>165</forces_angle_tolerance>
+            <update_rate>60</update_rate>
+            <grip_count_threshold>1</grip_count_threshold>
             <max_grip_count>20</max_grip_count>
-            <release_tolerance>0.00025</release_tolerance>
+            <release_tolerance>0.0004</release_tolerance>
             <disable_collisions_on_attach>false</disable_collisions_on_attach>
             <contact_topic>__default_topic__</contact_topic>

File: chessaton_description/urdf/chessaton_hand.xacro (robot description, xacro)
@@ -23,13 +23,13 @@
     		</collision>
             <inertial>
-                <origin xyz="-0.0266115313266715 -0.00796138911947138 -0.00177094547635764" rpy="0 0 0" />
-                <mass value="0.06585" />
+                <origin xyz="-0.02661 -0.0071 -0.001771" rpy="0 0 0" />
+                <mass value="0.066" />
                 <inertia
-                  ixx="1.94087633896407E-05"
-                  ixy="-4.40301296709736E-09"
-                  ixz="4.53529613378857E-07"
-                  iyy="9.16254031981619E-06"
-                  iyz="-1.54322487670811E-09"
-                  izz="2.20818336953172E-05" />
+                  ixx="1.9409E-05"
+                  ixy="-4.403E-09"
+                  ixz="4.5353E-07"
+                  iyy="9.1625E-06"
+                  iyz="-1.5432E-09"
+                  izz="2.2082E-05" />
             </inertial>
     	</link>
@@ -58,15 +58,15 @@
             <inertial>
                 <origin
-                  xyz="0.0127034645973708 0.00154565127207735 0.0030231093837057"
+                  xyz="0.012703 0.0015457 0.0030231"
                   rpy="0 0 0" />
                 <mass
                   value="0.006" />
                 <inertia
-                  ixx="8.35673086475568E-07"
-                  ixy="-1.33373055978949E-07"
-                  ixz="1.71871382347731E-07"
-                  iyy="1.12518172710191E-06"
-                  iyz="1.94898487683555E-07"
-                  izz="1.56282552281173E-06" />
+                  ixx="8.3567E-07"
+                  ixy="-1.3337E-07"
+                  ixz="1.7187E-07"
+                  iyy="1.1252E-06"
+                  iyz="1.949E-07"
+                  izz="1.5628E-06" />
             </inertial>
     	</link>
@@ -94,13 +94,13 @@
     		</collision>
             <inertial>
-                <origin xyz="0.0127037648728564 -0.00154618659083175 -0.00302306815560061" rpy="0 0 0" />
+                <origin xyz="0.012704 -0.0015462 -0.0030231" rpy="0 0 0" />
                 <mass value="0.006" />
                 <inertia
-                  ixx="8.35698479109993E-07"
-                  ixy="1.33368292398724E-07"
-                  ixz="-1.71864622126188E-07"
-                  iyy="1.1252213355056E-06"
-                  iyz="1.94907513457399E-07"
-                  izz="1.56288435175142E-06" />
+                  ixx="8.357E-07"
+                  ixy="1.3337E-07"
+                  ixz="-1.7186E-07"
+                  iyy="1.1252E-06"
+                  iyz="1.9491E-07"
+                  izz="1.5629E-06" />
             </inertial>
     	</link>
