Commit message: Modify: replaced main groups with chains and seperated virtual joint

File: chessaton_moveit_config/srdf/chessaton_macro.srdf.xacro (robot description, xacro)
@@ -12,22 +12,23 @@
         <!--SUBGROUPS- Groups can also be formed by referencing to already defined group names-->
         <group name="chessaton_arm">
-            <joint name="chessaton_joint1"/>
-            <joint name="virtual_joint"/>
-            <joint name="chessaton_joint2"/>
-            <joint name="chessaton_joint3"/>
-            <joint name="chessaton_joint4"/>
+            <chain base_link="chessaton_link0" tip_link="chessaton_link4"/>
         </group>
+        <!--GROUP STATES- Purpose- Define a named state for a particular group, in terms of joint values. This is useful to define states like 'folded arms'-->
+        <group_state group="chessaton_arm" name="all_zero">
+            <joint name="chessaton_joint1" value="0" />
+            <joint name="chessaton_joint2" value="0" />
+            <joint name="chessaton_joint3" value="0" />
+            <joint name="chessaton_joint4" value="0" />
+        </group_state>
+        <!--VIRTUAL JOINT= Purpose= this element defines a virtual joint between a robot link and an external frame of reference (considered fixed with respect to the robot)-->
+        <virtual_joint child_link="chessaton_link0" name="virtual_joint" parent_frame="world" type="fixed"/>
         <group name="chessaton_hand">
             <link name="chessaton_gripper"/>
             <link name="left_finger"/>
             <link name="right_finger"/>
+            <joint name="left_finger_joint"/>
+            <joint name="right_finger_joint"/>
         </group>
         <!--GROUP STATES- Purpose- Define a named state for a particular group, in terms of joint values. This is useful to define states like 'folded arms'-->
-        <group_state name="base_pose" group="chessaton_arm">
-            <joint name="chessaton_joint1" value="0"/>
-            <joint name="chessaton_joint2" value="0"/>
-            <joint name="chessaton_joint3" value="0"/>
-            <joint name="chessaton_joint4" value="0"/>
-        </group_state>
         <group_state name="hand_close" group="chessaton_hand">
             <joint name="left_finger_joint" value="0"/>
@@ -38,4 +39,8 @@
             <joint name="right_finger_joint" value="-0.03"/>
         </group_state>
+        <group name="chessaton_arm_hand">
+            <group name="chessaton_arm"/>
+            <group name="chessaton_hand"/>
+        </group>
         <!--END EFFECTOR- Purpose- Represent information about an end effector.-->
         <end_effector name="chessaton_hand" parent_link="chessaton_link4" group="chessaton_hand" parent_group="chessaton_arm"/>

Commit message: Add: add home position for arm_hand group

File: chessaton_moveit_config/srdf/chessaton_macro.srdf.xacro (robot description, xacro)
@@ -12,5 +12,5 @@
         <!--SUBGROUPS- Groups can also be formed by referencing to already defined group names-->
         <group name="chessaton_arm">
-            <chain base_link="chessaton_link0" tip_link="chessaton_link4"/>
+            <chain base_link="chessaton_link0" tip_link="chessaton_hand_tcp"/>
         </group>
         <!--GROUP STATES- Purpose- Define a named state for a particular group, in terms of joint values. This is useful to define states like 'folded arms'-->
@@ -20,4 +20,6 @@
             <joint name="chessaton_joint3" value="0" />
             <joint name="chessaton_joint4" value="0" />
+            <joint name="chessaton_hand_tcp_roll_virtual_joint" value="0" />
+            <joint name="chessaton_hand_tcp_yaw_virtual_joint" value="0" />
         </group_state>
         <!--VIRTUAL JOINT= Purpose= this element defines a virtual joint between a robot link and an external frame of reference (considered fixed with respect to the robot)-->
@@ -27,4 +29,5 @@
             <link name="left_finger"/>
             <link name="right_finger"/>
+            <!-- <link name="chessaton_hand_tcp"/> -->
             <joint name="left_finger_joint"/>
             <joint name="right_finger_joint"/>
@@ -43,6 +46,16 @@
             <group name="chessaton_hand"/>
         </group>
+        <group_state group="chessaton_arm_hand" name="home">
+            <joint name="chessaton_joint1" value="0" />
+            <joint name="chessaton_joint2" value="0" />
+            <joint name="chessaton_joint3" value="0" />
+            <joint name="chessaton_joint4" value="0" />
+            <joint name="chessaton_hand_tcp_roll_virtual_joint" value="0" />
+            <joint name="chessaton_hand_tcp_yaw_virtual_joint" value="0" />
+            <joint name="left_finger_joint" value="0"/>
+            <joint name="right_finger_joint" value="0"/>
+        </group_state>
         <!--END EFFECTOR- Purpose- Represent information about an end effector.-->
-        <end_effector name="chessaton_hand" parent_link="chessaton_link4" group="chessaton_hand" parent_group="chessaton_arm"/>
+        <end_effector name="chessaton_hand" parent_link="chessaton_hand_tcp" group="chessaton_hand" parent_group="chessaton_arm"/>
         <!--DISABLE COLLISIONS- By default it is assumed that any link of the robot could potentially come into collision with any other link in the robot. This tag disables collision checking between a specified pair of links. -->
         <disable_collisions link1="chessaton_gripper" link2="chessaton_link3" reason="Never"/>
@@ -61,4 +74,8 @@
         <disable_collisions link1="chessaton_link4" link2="right_finger" reason="Never"/>
         <disable_collisions link1="left_finger" link2="right_finger" reason="Never"/>
+        <disable_collisions link1="chessaton_hand_tcp_roll" link2="left_finger" reason="Never"/>
+        <disable_collisions link1="chessaton_hand_tcp_roll" link2="right_finger" reason="Never"/>
+        <disable_collisions link1="chessaton_hand_tcp_yaw" link2="left_finger" reason="Never"/>
+        <disable_collisions link1="chessaton_hand_tcp_yaw" link2="right_finger" reason="Never"/>
     </xacro:macro>
 </robot>

Commit message: Modify: decrease speed of movements

File: chessaton_moveit_config/srdf/chessaton_macro.srdf.xacro (robot description, xacro)
@@ -39,6 +39,6 @@
         </group_state>
         <group_state name="hand_open" group="chessaton_hand">
-            <joint name="left_finger_joint" value="0.023"/>
-            <joint name="right_finger_joint" value="-0.023"/>
+            <joint name="left_finger_joint" value="0.02"/>
+            <joint name="right_finger_joint" value="-0.02"/>
         </group_state>
         <group name="chessaton_arm_hand">
